Commit message: robot

File: description/robot_core.xacro (robot description, xacro)
@@ -1 +1,160 @@
-<!-- #hi this place is for you to define the robo property -->
+<?xml version="1.0"?>
+<robot xmlns:xacro="http://www.ros.org/wiki/xacro" name="robot">
+	<xacro:include filename="inertial_macros.xacro" />
+	<!-- color and textures -->
+	<material name="white">
+		<color rgba="1 1 1 1" />
+	</material>
+	<material name="orange">
+		<color rgba="1 .3 .1 1" />
+	</material>
+	<material name="blue">
+		<color rgba=".2 .2 1 1" />
+	</material>
+	<material name="black">
+		<color rgba="0 0 0 1" />
+	</material>
+	<!-- base link -->
+	<link name="base_link">
+	</link>
+	<!-- BASE_FOOTPRINT LINK -->
+        <joint name="base_footprint_joint" type="fixed">
+	    <parent link="base_link"/>
+	    <child link="base_footprint"/>
+	    <origin xyz="0 0 0" rpy="0 0 0"/>
+        </joint>
+        <link name="base_footprint">
+        </link>
+	<!-- chassis link -->
+	<joint name="chassis_joint" type="fixed">
+		<parent link="base_link"/>
+		<child link="chassis"/>
+		<origin xyz="-0.1 0 0"/>
+	</joint>
+	<link name="chassis">
+		<visual>
+			<origin xyz =".15 0 0.075"/>
+			<geometry>
+				<box size="0.3 0.3 .15"/>
+			</geometry>
+			<material name="white"/>
+		</visual>
+		<collision>
+			<origin xyz =".15 0 0.075"/>
+			<geometry>
+				<box size="0.3 0.3 .15"/>
+			</geometry>
+		</collision>
+		<xacro:inertial_box mass="0.5" x="0.3" y="0.3" z="0.15">
+			<origin xyz="0.15 0 0.075" rpy="0 0 0"/>
+		</xacro:inertial_box>
+	</link>
+	<gazebo reference="chassis">
+		<material>Gazebo/White</material>
+	</gazebo>
+	<!-- left wheel -->
+	<joint name="left_wheel_joint" type="continuous">
+		<parent link="base_link"/>
+		<child link="left_wheel"/>
+		<origin xyz="-0.05 0.175 0" rpy="-${pi/2} 0 0" />
+		<axis  xyz="0 0 1"/>
+	</joint>
+	<link name="left_wheel">
+		<visual>
+			<geometry>
+				<cylinder radius="0.05" length="0.04"/>
+			</geometry>
+			<material name="blue"/>
+		</visual>
+		<collision>
+			<geometry>
+				<cylinder radius="0.05" length="0.04"/>
+			</geometry>
+		</collision>
+		<xacro:inertial_cylinder mass="0.1" length="0.04" radius="0.05">
+			<origin xyz="0 0 0" rpy="0 0 0"/>
+		</xacro:inertial_cylinder>
+	</link>
+	<gazebo reference="left_wheel">
+		<material>Gazebo/Black</material>
+	</gazebo>
+	<!-- right wheel -->
+	<joint name="right_wheel_joint" type="continuous">
+		<parent link="base_link"/>
+		<child link="right_wheel"/>
+		<origin xyz="-0.05 -0.175 0" rpy="${pi/2} 0 0" />
+		<axis  xyz="0 0 -1"/>
+	</joint>
+	<link name="right_wheel">
+		<visual>
+			<geometry>
+				<cylinder radius="0.05" length="0.04"/>
+			</geometry>
+			<material name="blue"/>
+		</visual>
+		<collision>
+			<geometry>
+				<cylinder radius="0.05" length="0.04"/>
+			</geometry>
+		</collision>
+		<xacro:inertial_cylinder mass="0.1" length="0.04" radius="0.05">
+			<origin xyz="0 0 0" rpy="0 0 0"/>
+		</xacro:inertial_cylinder>
+	</link>
+	<gazebo reference="right_wheel">
+		<material>Gazebo/Black</material>
+	</gazebo>
+	<!-- caster wheel boys -->
+	<joint name="cw_right_joint" type="fixed">
+		<parent link="chassis"/>
+		<child link="cw_right"/>
+		<origin xyz=".25 -0.175 0" rpy="${pi/2} 0 0" />
+	</joint>
+	<link name="cw_right">
+		<visual>
+			<geometry>
+				<cylinder radius="0.05" length="0.04"/>
+			</geometry>
+			<material name="blue"/>
+		</visual>
+		<collision>
+			<geometry>
+				<cylinder radius="0.05" length="0.04"/>
+			</geometry>
+		</collision>
+		<xacro:inertial_cylinder mass="0.1" length="0.04" radius="0.05">
+			<origin xyz="0 0 0" rpy="0 0 0"/>
+		</xacro:inertial_cylinder>
+	</link>
+	<gazebo reference="cw_right">
+		<material>Gazebo/Black</material>
+		<mu1 value="0.001" />
+		<mu2 value="0.001" />
+	</gazebo>
+	<joint name="cw_left_joint" type="fixed">
+		<parent link="chassis"/>
+		<child link="cw_left"/>
+		<origin xyz=".25 0.175 0" rpy="${pi/2} 0 0" />
+	</joint>
+	<link name="cw_left">
+		<visual>
+			<geometry>
+				<cylinder radius="0.05" length="0.04"/>
+			</geometry>
+			<material name="blue"/>
+		</visual>
+		<collision>
+			<geometry>
+				<cylinder radius="0.05" length="0.04"/>
+			</geometry>
+		</collision>
+		<xacro:inertial_cylinder mass="0.1" length="0.04" radius="0.05">
+			<origin xyz="0 0 0" rpy="0 0 0"/>
+		</xacro:inertial_cylinder>
+	</link>
+	<gazebo reference="cw_left">
+		<material>Gazebo/Black</material>
+		<mu1 value="0.001" />
+		<mu2 value="0.001" />
+	</gazebo>
+</robot>
